File: PCB layout.sch (KiCad schematic (older format))
At the start: 14 parts, among them J2 Conn_01x02_Male, Q1 2P222

Commit message: Version 1.1
Parts:
- removed J2: Conn_01x02_Male, Connector_JST:JST_PH_S2B-PH-K_1x02_P2.00mm_Horizontal, symbol Connector:Conn_01x02_Male
- added JP2: HEADER-1X570MIL, Adafruit RFM+LoRa Breakout:1X05_ROUND_70, symbol Adafruit_RFM+LoRa_Breakout-eagle-import:HEADER-1X570MIL
- added RBAT1: 100K, Adafruit RFM+LoRa Breakout:0805-NO, symbol Device:R
- added RBAT2: 27K, Adafruit RFM+LoRa Breakout:0805-NO, symbol Device:R
- R1, R2, R3, R4, R_BJT1: footprint Resistor_THT:R_Axial_DIN0411_L9.9mm_D3.6mm_P12.70mm_Horizontal -> Adafruit RFM+LoRa Breakout:0805-NO
- Si7021: renamed from JP2; footprint Adafruit RFM+LoRa Breakout:1X05_ROUND_70 -> TerminalBlock_Altech:Altech_AK300_1x05_P5.00mm_45-Degree; symbol Adafruit_RFM+LoRa_Breakout-eagle-import:HEADER-1X570MIL -> PCB-layout-rescue:HEADER-1X570MIL-Adafruit_Si7021_Humidity-eagle-import
Connections:
- net labels added: +3V3, SCL, SDA
- wire segments 115 -> 129
Other:
- moved on the sheet: B1, GPSCONNECT1, Q1, R1, R2, R3, R4, R_BJT1, SENSOR1, SENSOR2, SENSOR3, SENSOR4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
